File: BDR.sch (KiCad schematic (older format))
At the start: 9 parts

Commit message: added ideal diode between BCR/BDR. Replaced load switch with ideal diode in inhibit switch circuit
Connections:
- new net: R?.~, R?.~, U?.12 (FB)
Changed lines of the file:
@@
 $Descr A4 11693 8268
 encoding utf-8
-Sheet 34 34
+Sheet 34 36
 Title ""
 Date ""

Commit message: Addded first portion of battery heater. Contains the temperature sensor and resistive heater. Need to add logic if it will be driven by OBC.
Connections:
- new net: R?.~, R?.~, U?.12 (FB)
Changed lines of the file:
@@
 EESchema Schematic File Version 4
 LIBS:Main-cache
-EELAYER 29 0
+EELAYER 26 0
 EELAYER END
 $Descr A4 11693 8268
 encoding utf-8
-Sheet 34 36
+Sheet 34 37
 Title ""
 Date ""
