File: Main.sch (KiCad schematic (older format))
At the start: 75 parts, among them SW1 SW_Push, U2 MSP430F5529IPN, U3 TPS2557, U4 TPS2557, U5 TPS2557, U6 TPS2557

Commit message: Added MSP430 to main
Parts:
- removed C1, C2, C3, C4: 0.1u, symbol Main-rescue:C-Device
- removed C5, C6, C7, C8: 150u, symbol Main-rescue:C-Device
- removed R10, R11, R12, R9: TBD, symbol Main-rescue:R_Shunt-Device
- removed R13, R14, R15, R16: R, symbol Main-rescue:R-Device
- removed U2: MSP430F5529IPN, PN80, symbol Main-rescue:MSP430F5529IPN-MSP430
- removed U3, U4, U5, U6: TPS2557, symbol Main-rescue:TPS2557-CustomSymbols
- M? (x2): symbol pspice:MNMOS -> Main-rescue:MNMOS-pspice
Connections:
- net labels removed: ACS, OBC, PAYLOAD, RF
- wire segments 296 -> 313
- no-connect marks 9 -> 1
