File: SPV1040.sch (KiCad schematic (older format))
At the start: 10 parts

Commit message: finish
Parts:
- removed C? (x2): 100u, symbol Main-rescue:C-Device
- removed C? (x2): 1n, symbol Device:C
- removed L?: 10uH, symbol Main-rescue:L-Device
- removed R?: 1k, symbol Main-rescue:R-Device
- removed R?: 768k, symbol Device:R
- removed R?: 330k, symbol Device:R
- removed SC?: Solar_Cell, symbol Device:Solar_Cell
- removed U?: SPV1040, symbol Main-rescue:SPV1040-CustomSymbols
Other:
- note removed: "Inductor:\nB82442T1103K050"
